File: pcb/button_pullup.kicad_sch (KiCad schematic)
At the start: 4 parts, among them SW2 SW_Push

Commit message: rework to tia feedback selection, board power, and ui
Parts:
- renumbered C56 to C59, R33 to R39, R34 to R40
