File: pcb/button_pullup.kicad_sch (KiCad schematic)
At the start: 4 parts, among them SW2 SW_Push

Commit message: chore: many changes checkpoint
Parts:
- removed C59: 100n, symbol Device:C
- removed R39, R40: 10k, symbol Device:R
- removed SW2: SW_Push, symbol Switch:SW_Push
- added SW2: SW_Push, project_library:SWT0310-043016GSA, symbol project_library:SW_Push
Connections:
- net BUT: now also SW2.1
- net GND: now also SW2.2
