File: pcb/microcontroller.kicad_sch (KiCad schematic)
At the start: 19 parts, among them J1 Conn_01x04_Pin, J2 USB_C_Receptacle_USB2.0_16P, SW1 SW_Push, U17 ATSAMD21G18A, Y1 32.786

Commit message: rework to tia feedback selection, board power, and ui
Other:
- removed sheet ui
