File: pcb/microcontroller.kicad_sch (KiCad schematic)
At the start: 19 parts, among them J1 Conn_01x04_Pin, J2 USB_C_Receptacle_USB2.0_16P, SW1 SW_Push, U17 ATSAMD21G18A, Y1 32.786

Commit message: chore: many changes checkpoint
Parts:
- removed C55: 10u, symbol Device:C
- removed J2: USB_C_Receptacle_USB2.0_16P, symbol Connector:USB_C_Receptacle_USB2.0_16P
- removed SW1: SW_Push, symbol Switch:SW_Push
- added C77: 10u, Capacitor_Tantalum_SMD:CP_EIA-3528-12_Kemet-T, symbol Device:C_Polarized
- added C89: 100n, Capacitor_SMD:C_0603_1608Metric, symbol Device:C
- added D12: SMAJ5.0A, Diode_SMD:D_SMA, symbol Diode:SMAJ5.0A
- added F2: Polyfuse, Fuse:Fuse_1812_4532Metric, symbol Device:Polyfuse
- added FB4: FerriteBead, Inductor_SMD:L_0603_1608Metric, symbol Device:FerriteBead
- added J2: USB_C_PROG, project_library:USB4110-GF-A, symbol project_library:USB_C_PROG
- added SW1: SW_Push, project_library:SWT0310-043016GSA, symbol project_library:SW_Push
- C47, C48, C49, C50, C51, C52, C53, C54: footprint (none) -> Capacitor_SMD:C_0603_1608Metric
- J1: footprint (none) -> Connector:FanPinHeader_1x04_P2.54mm_Vertical
- R28, R29, R30, R31, R32: footprint (none) -> Resistor_SMD:R_0603_1608Metric
- U17: footprint ATSAMD21G18A-AU:QFP50P900X900X120-48N -> Package_QFP:TQFP-48_7x7mm_P0.5mm
- Y1: footprint (none) -> Crystal:Crystal_AT310_D3.0mm_L10.0mm_Horizontal
Connections:
- net +5VUSB: now also C77.1, C89.2, FB4.2
- net GND: now also C77.2, C89.1, D12.2 (A2), J2.A1 (GND), J2.A12 (GND), J2.B1 (GND), J2.B12 (GND), J2.S1 (SHIELD), SW1.1
- net at R32.1: now also J2.A6 (D+), J2.B6 (D+)
- net at R29.1: now also J2.A5 (CC1)
- net at R31.1: now also J2.A7 (D-), J2.B7 (D-)
- net at R30.1: now also J2.B5 (CC2)
- net at R28.2, U17.40 (~{RESETN}): now also SW1.2
- net +3.3VD renamed +3.3VMCU
- net +3.3VMCU: no longer C54.1, R28.1
- new net: F2.1, J2.A4 (VBUS), J2.A9 (VBUS), J2.B4 (VBUS), J2.B9 (VBUS)
- new net: D12.1 (A1), F2.2, FB4.1
- new net +3V3MCU: C54.1, R28.1
- no-connect marks 2 -> 34
Other:
- note removed: "need a way to switch source for programming board"
- moved on the sheet: C48, C51, C53, C54, J1, R28, R29, R30, R31, R32, Y1
