File: pcb/digital_isolation.kicad_sch (KiCad schematic)
At the start: 10 parts, among them U19 ISO7740, U21 ISO7740, U22 ISO7742

Commit message: chore: many changes checkpoint
Parts:
- removed C71, C79: 100n, symbol Device:C
- removed U19, U21: ISO7740, DBQ0016A_N, symbol project_library:ISO7740
- removed U22: ISO7742, DBQ0016A_N, symbol project_library:ISO7742
- added C63, C64: 100n, Capacitor_SMD:C_0603_1608Metric, symbol Device:C
- added U11, U9: ISO7740, Package_SO:SSOP-16_3.9x4.9mm_P0.635mm, symbol project_library:ISO7740
- added U19: ISO7742, Package_SO:SSOP-16_3.9x4.9mm_P0.635mm, symbol project_library:ISO7742
- C37, C69, C70, C78: footprint (none) -> Capacitor_SMD:C_0603_1608Metric
- R48: footprint (none) -> Resistor_SMD:R_0603_1608Metric
Connections:
- net ISO_EN is gone; now on net EN: R48.1
- net +5VA: now also C63.1, C64.1, U11.16 (VCC2), U19.16 (VCC2), U9.16 (VCC2); no longer C37.1
- net ADC_CS: now also U9.4 (INB)
- net DAC_CS: now also U9.3 (INA)
- net DRDY: now also U19.6 (OUTD)
- net EN: now also U11.10 (EN2), U19.10 (EN2), U19.7 (EN1), U9.10 (EN2)
- net GND: now also C37.1, C70.1, U11.2 (GND1), U11.8 (GND1), U19.2 (GND1), U19.8 (GND1), U9.2 (GND1), U9.6 (IND), U9.8 (GND1)
- net GNDA: now also C63.2, C64.2, U11.15 (GND2), U11.9 (GND2), U19.15 (GND2), U19.9 (GND2), U9.15 (GND2), U9.9 (GND2); no longer C37.2, C70.1
- net ISO_ADC_CS: now also U9.13 (OUTB)
- net ISO_DAC_CS: now also U9.14 (OUTA)
- net ISO_DRDY: now also U19.11 (IND)
- net ISO_MISO: now also U19.12 (INC)
- net ISO_MOSI: now also U19.13 (OUTB)
- net ISO_SCLK: now also U19.14 (OUTA)
- net MISO: now also U19.5 (OUTC)
- net MOSI: now also U19.4 (INB)
- net SCLK: now also U19.3 (INA)
- net ~{FBSA}: now also U11.6 (IND)
- net ~{FBSB}: now also U11.3 (INA)
- net ~{FBSC}: now also U11.4 (INB)
- net ~{FBSD}: now also U11.5 (INC)
- net ~{ISO_FBSA}: now also U11.11 (OUTD)
- net ~{ISO_FBSB}: now also U11.14 (OUTA)
- net ~{ISO_FBSC}: now also U11.13 (OUTB)
- net ~{ISO_FBSD}: now also U11.12 (OUTC)
- net +3.3V renamed +3V3
- net +3V3: now also C37.2, U11.1 (VCC1), U19.1 (VCC1), U9.1 (VCC1)
- no-connect marks 3 -> 5
Other:
- moved on the sheet: C78, R48
