File: pcb/dual_rail_variable_psu.kicad_sch (KiCad schematic)
At the start: 22 parts, among them U15 OPA140, U16 OPA1611, U4 OPA1611, U8 DAC8551

Commit message: chore: many changes checkpoint
Parts:
- removed unit 1 of U4
- added U18: OPA1611, Package_SO:SOIC-8_3.9x4.9mm_P1.27mm, symbol project_library:OPA1611
- C13, C15, C16, C32, C42, C43, C44, C45, C46: footprint (none) -> Capacitor_SMD:C_0603_1608Metric
- R1, R18, R20, R27, R4, R7, R9: footprint (none) -> Resistor_SMD:R_0603_1608Metric
- R11: value 1k -> 10k; footprint (none) -> Resistor_SMD:R_0603_1608Metric
- R19: value 2k -> 20k; footprint (none) -> Resistor_SMD:R_0603_1608Metric
- U15: footprint DBV5 -> Package_TO_SOT_SMD:SOT-23-5
- U16, U4: footprint D0008A_N -> Package_SO:SOIC-8_3.9x4.9mm_P1.27mm
- U8: footprint DGK8 -> Package_SO:VSSOP-8_3x3mm_P0.65mm
Connections:
- net +12VA: now also U18.7
- net -12VA: now also U18.4
- net V_DAC_FILTERED: now also U18.3 (+)
- net at R1.1, R9.2: now also U18.6
- net at R1.2, R4.1: now also U18.2 (-)
- no-connect marks 3 -> 6
