File: pcb/encoder_layout.kicad_sch (KiCad schematic)
At the start: 10 parts

Commit message: chore: many changes checkpoint
Parts:
- removed R37: 10k, symbol Device:R
- added R43: 10k, Resistor_SMD:R_0603_1608Metric, symbol Device:R
- C56, C57, C58: footprint (none) -> Capacitor_SMD:C_0603_1608Metric
- MT1: footprint PEC11R-4215F-S0024:XDCR_PEC11R-4215F-S0024 -> project_library:PEC11R
- R33, R34, R35, R36, R38: footprint (none) -> Resistor_SMD:R_0603_1608Metric
Connections:
- net BUT: now also R33.2; no longer R33.1
- net at MT1.1, R34.1: now also R33.1; no longer R33.2
- net at MT1.B, R36.1: now also R43.1; no longer R35.1
- net at MT1.A, R38.2: now also R35.1
- net +3.3V renamed +3V3
- net +3V3: now also R43.2
Other:
- moved on the sheet: C56, C57, R36, R38
