File: pcb/photoelectric_effect_demonstrator.kicad_sch (KiCad schematic)
At the start: 0 parts

Commit message: chore: many changes checkpoint
Connections:
- no-connect marks 0 -> 27
Other:
- added sheet logic_stepup (logic_stepup.kicad_sch)
- sheet adc ports: added ~{DRDY}; removed DDRY
- sheet mcu_pin_fanout ports: added FBSBA, FBSBB, FBSBC, ~{FBSA}, ~{FBSB}, ~{FBSC}, ~{FBSD}, ~{FBSE}, ~{FBSF}; removed none
- sheet phototube_instrumentation ports: added C_TUBE_OUT, REF_SEL, V_TUBE_OUT; removed C_TUBE, V_TUBE
- sheet ui ports: added A0, BR1, BR2, BSA, BSB, CS, EN1A, EN1B, EN1BUT, EN2A, EN2B, EN2BUT, MOSI, PWM, RST, SCLK; removed none
- note added: "NOT ISOLATED"
