File: pcb/phototube_instrumentation.kicad_sch (KiCad schematic)
At the start: 25 parts, among them U11 OPA1612AxD, U12 OPA140, U6 OPA140, U6 OPA1612AxD, U9 OPA1612AxD

Commit message: chore: many changes checkpoint
Parts:
- removed C41: 100n, symbol Device:C
- removed U11, U6, U9: OPA1612AxD, symbol Amplifier_Operational:OPA1612AxD
- removed U6: OPA140, DBV5, symbol project_library:OPA140
- added C29: 100n, Capacitor_SMD:C_0603_1608Metric, symbol Device:C
- added U26: OPA140, Package_TO_SOT_SMD:SOT-23-5, symbol project_library:OPA140
- added U6: OPA1612, Package_SO:SOIC-8_3.9x4.9mm_P1.27mm, symbol project_library:OPA1612
- C20, C21, C22, C26, C27, C38, C40: footprint (none) -> Capacitor_SMD:C_0603_1608Metric
- R10: value 3k -> 30k; footprint (none) -> Resistor_SMD:R_0603_1608Metric
- R12, R23: value 2k -> 20k; footprint (none) -> Resistor_SMD:R_0603_1608Metric
- R13: value 1k -> 10k; footprint (none) -> Resistor_SMD:R_0603_1608Metric
- R14, R15, R16, R22, R24, R25, R26: footprint (none) -> Resistor_SMD:R_0603_1608Metric
- U12: footprint DBV5 -> Package_TO_SOT_SMD:SOT-23-5
Connections:
- net +12VA: now also C27.2, C29.1, U26.5, U6.8 (V+); no longer C26.2
- net -12VA: now also C26.2, U26.2, U6.4 (V-); no longer C27.2
- net FEED_IN: now also D1.2 (A), R26.2, U12.3 (+); no longer R14.1
- net FEED_OUT: now also R14.1, U12.1; no longer D1.2 (A), R26.2
- net GNDA: now also U12.4 (-), C29.2
- net TUBE_CA: now also U26.3 (+); no longer U12.3 (+)
- net V_TIA_OFSET: now also U6.1
- net V_TUBE: now also U26.1, U26.4 (-); no longer R25.2, U12.1, U12.4 (-)
- net V_TUBE_OFSET: now also U6.7
- net at C20.1, R14.2, R15.1: now also U6.2 (-)
- net at C38.1, R16.2, R24.1: now also U6.6 (-)
- net at R13.2, R23.1: now also U6.5 (+)
- net at R10.1, R12.2: now also U6.3 (+)
- net C_TUBE renamed C_TUBE_OUT
- new net V_TUBE_OUT: R25.2
Other:
- added sheet relay5 (relay.kicad_sch)
- note added: "NEEDS FOOTPRINT"
- moved on the sheet: C20, C38, C40, D1, R10, R12, R13, R14, R15, R16, R22, R23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
