File: pcb/reference_voltage.kicad_sch (KiCad schematic)
At the start: 3 parts, among them U5 LTC6655

Commit message: chore: many changes checkpoint
Parts:
- C24, C25: footprint (none) -> Capacitor_SMD:C_0201_0603Metric
- U5: footprint 05-08-1660_ADI -> Package_SO:MSOP-8_3x3mm_P0.65mm
