File: pcb/tia_feedback_select.kicad_sch (KiCad schematic)
At the start: 15 parts, among them U14 ADG1211YRUZ-REEL7

Commit message: chore: many changes checkpoint
Parts:
- removed C63: 47p, symbol Device:C
- removed C64: 470p, symbol Device:C
- removed U14: ADG1211YRUZ-REEL7, RU_16_ADI, symbol project_library:ADG1211YRUZ-REEL7
- added C30: 100n, Capacitor_SMD:C_0603_1608Metric, symbol Device:C
- added C41: 47p, Capacitor_SMD:C_0603_1608Metric, symbol Device:C
- added R59, R60, R62, R74: 10k, Resistor_SMD:R_0603_1608Metric, symbol Device:R
- added U10: ADG1211, Package_SO:TSSOP-16_4.4x5mm_P0.65mm, symbol project_library:ADG1211
- C19, C33, C34, C35, C65: footprint (none) -> Capacitor_SMD:C_0603_1608Metric
- C36: value 100n -> 470p; footprint (none) -> Capacitor_SMD:C_0603_1608Metric
- R17, R5, R51, R56, R6, R61: footprint (none) -> Resistor_SMD:R_0603_1608Metric
Connections:
- net +12VA: now also U10.13 (VDD)
- net -12VA: now also C30.1, U10.4 (VSS); no longer C36.2
- net FIN: now also U10.11 (S3), U10.14 (S2), U10.3 (S1), U10.6 (S4)
- net FOUT: now also C36.1, C41.1
- net GNDA: now also C30.2, U10.5 (GND); no longer C36.1
- net relay1/D: now also C36.2
- net ~{FBSA}: now also R62.2, U10.1 (IN1)
- net ~{FBSB}: now also R59.2, U10.16 (IN2)
- net ~{FBSC}: now also R60.2, U10.9 (IN3)
- net ~{FBSD}: now also R74.2, U10.8 (IN4)
- net at C33.2, R5.2: now also U10.2 (D1)
- net at R51.2: now also C41.2, U10.7 (D4)
- net at C34.2, R6.2: now also U10.15 (D2)
- net at C35.2, R17.2: now also U10.10 (D3)
- new net +5VA: R59.1, R60.1, R62.1, R74.1
Other:
- moved on the sheet: C19
