File: pcb/usbc_psu.kicad_sch (KiCad schematic)
At the start: 12 parts, among them J3 USB_C_Receptacle_USB2.0_16P, U23 TLV75533PDBV

Commit message: chore: many changes checkpoint
Parts:
- removed C77, C84: 100n, symbol Device:C
- removed C80: 10u, symbol Device:C
- removed J3: USB_C_Receptacle_USB2.0_16P, symbol Connector:USB_C_Receptacle_USB2.0_16P
- removed U23: TLV75533PDBV, Package_TO_SOT_SMD:SOT-23-5, symbol Regulator_Linear:TLV75533PDBV
- added C71, C72, C73, C87: 100n, Capacitor_SMD:C_0603_1608Metric, symbol Device:C
- added C74, C75: 10u, Capacitor_Tantalum_SMD:CP_EIA-3528-12_Kemet-T, symbol Device:C_Polarized
- added D11, D13: SS14, Diode_SMD:D_SMA, symbol Diode:SS14
- added J3: USB_C_PWR, project_library:USB4135-GF-A, symbol project_library:USB_C_PWR
- added Q14: AO3401A, Package_TO_SOT_SMD:SOT-23, symbol Transistor_FET:AO3401A
- added R73: 100k, Resistor_SMD:R_0603_1608Metric, symbol Device:R
- added U23, U24: TLV75533PDBVR, project_library:SOT95P280X145-5N, symbol project_library:TLV75533PDBVR
- C81: footprint (none) -> Capacitor_Tantalum_SMD:CP_EIA-3528-12_Kemet-T
- C82: footprint (none) -> Capacitor_SMD:C_0201_0603Metric
- F1: footprint (none) -> Fuse:Fuse_1812_4532Metric
- FB5: footprint (none) -> Inductor_SMD:L_0603_1608Metric
- R67, R68: footprint (none) -> Resistor_SMD:R_0603_1608Metric
Connections:
- net +3V3: now also C72.2, C74.1, U23.5 (OUT)
- net +5V: now also C73.2, D13.2 (A), Q14.1 (G), R73.1, U23.1 (IN), U23.3 (EN)
- net GND: now also C71.1, C72.1, C73.1, C74.2, C75.2, C87.1, J3.A12 (GND), J3.B12 (GND), J3.S1 (SHIELD), J3.S2 (SHIELD), J3.S3 (SHIELD), J3.S4 (SHIELD), R73.2, U23.2 (GND), U24.2 (GND)
- net at F1.1: now also J3.A9 (VBUS), J3.B9 (VBUS)
- net at R67.1: now also J3.A5 (CC1)
- net at R68.1: now also J3.B5 (CC2)
- new net: C71.2, D13.1 (K), Q14.2 (S), U24.1 (IN), U24.3 (EN)
- new net: D11.1 (K), Q14.3 (D)
- new net +3V3MCU: C75.1, C87.2, U24.5 (OUT)
- new net +5VUSB: D11.2 (A)
- no-connect marks 6 -> 0
Other:
- note added: "NEED FOOTPRINT CAP and FUSE"
- moved on the sheet: C81, C82, D7, F1, FB5, R67, R68
